Commit message: xacro namespace inserted to its flags, option --inorder inserted (these changes are required by the current version of xacro)

File: xacro/p3dx/pioneer3dx.xacro (robot description, xacro)
@@ -13,4 +13,5 @@
   <xacro:laser_gpu name="front_laser" parent="chassis" xyz="0.16 0 0.1" rpy="0 0 0" meshes="package://gazebo_plugins/test/multi_robot_scenario/meshes/laser" />
     -->
+  <!-- Camera -->
   <xacro:include filename="$(find p3dx_gazebo)/xacro/camera/camera.xacro"/>
   <xacro:cam name="front_camera" parent="chassis" xyz="0 0 0.5" rpy="0 0 0" />

File: xacro/p3dx/pioneer3dx_chassis.xacro (robot description, xacro)
@@ -1,5 +1,5 @@
 <?xml version="1.0"?>
 <robot xmlns:xacro="http://ros.org/wiki/xacro">
-  <property name="M_PI" value="3.1415926535897931" />
+  <xacro:property name="M_PI" value="3.1415926535897931" />
   <xacro:macro name="pioneer_chassis" params="name parent xyz rpy meshes">
   <!-- Chassis -->

File: xacro/p3dx/pioneer3dx_sonar.xacro (robot description, xacro)
@@ -1,5 +1,5 @@
 <?xml version="1.0"?>
 <robot xmlns:xacro="http://ros.org/wiki/xacro">
-  <property name="M_PI" value="3.1415926535897931" />
+  <xacro:property name="M_PI" value="3.1415926535897931" />
   <xacro:macro name="pioneer_sonar" params="name parent xyz rpy meshes">
   <!-- Front Sonar -->

File: xacro/p3dx/pioneer3dx_swivel.xacro (robot description, xacro)
@@ -1,5 +1,5 @@
 <?xml version="1.0"?>
 <robot xmlns:xacro="http://ros.org/wiki/xacro">
-  <property name="M_PI" value="3.1415926535897931" />
+  <xacro:property name="M_PI" value="3.1415926535897931" />
   <xacro:macro name="pioneer_swivel" params="parent xyz rpy meshes">
   <!-- Swivel -->

File: xacro/p3dx/pioneer3dx_wheel.xacro (robot description, xacro)
@@ -2,5 +2,5 @@
 <robot
   xmlns:xacro="http://ros.org/wiki/xacro">
-  <property name="M_PI" value="3.1415926535897931" />
+  <xacro:property name="M_PI" value="3.1415926535897931" />
   <xacro:macro name="pioneer_wheel" params="side parent xyz rpy radius meshes">
   <!-- Hubcap -->
@@ -29,5 +29,5 @@
       <origin xyz="0 0 0" rpy="0 0 0"/>
       <geometry>
-        <box size="0.01 0.01 0.01"/>
+        <box size="0.0001 0.0001 0.0001"/>
       </geometry>
     </collision>

Commit message: p3dx colors fixed

File: xacro/p3dx/pioneer3dx.xacro (robot description, xacro)
@@ -9,8 +9,7 @@
   <xacro:include filename="$(find p3dx_gazebo)/xacro/laser/hokuyo.xacro"/>
   <xacro:laser name="front_laser" parent="chassis" xyz="0.16 0 0.1" rpy="0 0 0" meshes="package://p3dx_gazebo/meshes/laser"/>
-  <!-- GPU Laser
-  <xacro:include filename="$(find gazebo_plugins)/test/multi_robot_scenario/xacro/laser/hokuyo_gpu.xacro"/>
-  <xacro:laser_gpu name="front_laser" parent="chassis" xyz="0.16 0 0.1" rpy="0 0 0" meshes="package://gazebo_plugins/test/multi_robot_scenario/meshes/laser" />
-    -->
+  <!-- GPU Laser -->
+<!--  <xacro:include filename="$(find gazebo_plugins)/test/multi_robot_scenario/xacro/laser/hokuyo_gpu.xacro"/>-->
+  <!--<xacro:laser_gpu name="front_laser2" parent="chassis" xyz="0.16 0 0.1" rpy="0 0 0" meshes="package://gazebo_plugins/test/multi_robot_scenario/meshes/laser" />-->
   <!-- Camera -->
   <xacro:include filename="$(find p3dx_gazebo)/xacro/camera/camera.xacro"/>

File: xacro/p3dx/pioneer3dx_sonar.xacro (robot description, xacro)
@@ -15,5 +15,6 @@
       <inertia ixx="1" ixy="0" ixz="0" iyy="1" iyz="0" izz="1"/>
     </inertial>
-    <visual name="front_sonar_vis">
+    <!--<visual name="front_sonar_vis">-->
+    <visual>
       <origin xyz="0 0 0" rpy="0 0 0"/>
       <geometry name="pioneer_geom">

File: xacro/p3dx/pioneer3dx_swivel.xacro (robot description, xacro)
@@ -19,5 +19,6 @@
       <inertia ixx="0.01" ixy="0" ixz="0" iyy="0.01" iyz="0" izz="0.01"/>
     </inertial>
-    <visual name="base_visual">
+    <!--<visual name="base_visual">-->
+    <visual>
       <origin xyz="0 0 0" rpy="0 0 0"/>
       <geometry name="pioneer_geom">
@@ -54,5 +55,6 @@
       <inertia ixx="0.012411765597" ixy="-0.000711733678" ixz="0.00050272983" iyy="0.015218160428" iyz="-0.000004273467" izz="0.011763977943"/>
     </inertial>
-    <visual name="base_visual">
+    <!--<visual name="base_visual">-->
+    <visual>
       <origin xyz="0 0 0" rpy="0 0 0"/>
       <geometry name="pioneer_geom">
@@ -86,5 +88,6 @@
       <inertia ixx="0.012411765597" ixy="-0.000711733678" ixz="0.00050272983" iyy="0.015218160428" iyz="-0.000004273467" izz="0.011763977943"/>
     </inertial>
-    <visual name="base_visual">
+    <!--<visual name="base_visual">-->
+    <visual>
       <origin xyz="0 0 0" rpy="0 0 0"/>
       <geometry name="pioneer_geom">

File: xacro/p3dx/pioneer3dx_wheel.xacro (robot description, xacro)
@@ -17,5 +17,6 @@
       <inertia ixx="0.012411765597" ixy="0" ixz="0" iyy="0.015218160428" iyz="0" izz="0.011763977943"/>
     </inertial>
-    <visual name="base_visual">
+    <!--<visual name="base_visual">-->
+    <visual>
       <origin xyz="0 0 0" rpy="0 0 0"/>
       <geometry name="pioneer_geom">
@@ -49,5 +50,6 @@
       <inertia ixx="0.012411765597" ixy="0" ixz="0" iyy="0.015218160428" iyz="0" izz="0.011763977943"/>
     </inertial>
-    <visual name="base_visual">
+    <!--<visual name="base_visual">-->
+    <visual>
       <origin xyz="0 0 0" rpy="0 0 0"/>
       <geometry name="pioneer_geom">
